Commit message: rotated lasers

File: src/robot_description/src/urdf/Floribot.urdf.xacro (robot description, xacro)
@@ -22,4 +22,5 @@
   <xacro:property name="rear_sensor_x" value="0.34" />
   <xacro:property name="camera_z" value="0.47" />
+  <xacro:property name="pi" value="3.141592653589793" />
   <link name="base_link">
     <visual>
@@ -311,5 +312,5 @@
     <parent link="front_wagon"/>
     <child link="front_laser_link"/>
-    <origin xyz="${front_sensor_x} 0 ${sensor_z}" rpy="0 0 0"/>
+    <origin xyz="${front_sensor_x} 0 ${sensor_z}" rpy="${pi} 0 0"/>
   </joint>
   <gazebo reference="front_laser_link">
@@ -367,5 +368,5 @@
     <parent link="rear_wagon"/>
     <child link="rear_laser_link"/>
-    <origin xyz="${rear_sensor_x} 0 ${sensor_z}" rpy="0 0 3.14159"/>
+    <origin xyz="${rear_sensor_x} 0 ${sensor_z}" rpy="${pi} 0 ${pi}"/>
   </joint>
   <gazebo reference="rear_laser_link">

Commit message: Update Floribot.urdf.xacro

File: src/robot_description/src/urdf/Floribot.urdf.xacro (robot description, xacro)
@@ -22,5 +22,5 @@
   <xacro:property name="rear_sensor_x" value="0.34" />
   <xacro:property name="camera_z" value="0.47" />
-  <xacro:property name="pi" value="3.141592653589793" />
+  <!-- <xacro:property name="pi" value="3.141592653589793" /> Muss nicht definiert werden. -->
   <link name="base_link">
     <visual>

Commit message: Update Floribot.urdf.xacro

File: src/robot_description/src/urdf/Floribot.urdf.xacro (robot description, xacro)
@@ -18,8 +18,9 @@
   <xacro:property name="horizontal_length" value="0.055" />
   <xacro:property name="wheel_joint_2_mid_joint" value="0.383" />
-  <xacro:property name="sensor_z" value="0.36" />
-  <xacro:property name="front_sensor_x" value="0.34" />
-  <xacro:property name="rear_sensor_x" value="-0.34" />
-  <xacro:property name="camera_z" value="0.47" />
+  <xacro:property name="sensor_z" value="0.03" />
+  <xacro:property name="front_sensor_x" value="0.3315" />
+  <xacro:property name="rear_sensor_x" value="-0.3315" />
+  <xacro:property name="camera_z" value="0.263" />
+  <xacro:property name="camera_angle" value="0.6" />
   <!-- <xacro:property name="pi" value="3.141592653589793" /> Muss nicht definiert werden. -->
   <link name="base_link">
@@ -310,5 +311,5 @@
   </link>
   <joint name="front_laser_joint" type="fixed">
-    <parent link="front_wagon"/>
+    <parent link="axesFront"/>
     <child link="front_laser_link"/>
     <origin xyz="${front_sensor_x} 0 ${sensor_z}" rpy="${pi} 0 0"/>
@@ -366,5 +367,5 @@
   </link>
   <joint name="rear_laser_joint" type="fixed">
-    <parent link="rear_wagon"/>
+    <parent link="axesRear"/>
     <child link="rear_laser_link"/>
     <origin xyz="${rear_sensor_x} 0 ${sensor_z}" rpy="${pi} 0 ${pi}"/>
@@ -422,7 +423,7 @@
   </link>
   <joint name="front_camera_joint" type="fixed">
-    <parent link="front_wagon"/>
+    <parent link="base_link"/>
     <child link="front_camera_link"/>
-    <origin xyz="${front_sensor_x} 0 ${camera_z}" rpy="0 0 0"/>
+    <origin xyz="${front_sensor_x} 0 ${camera_z}" rpy="0 ${camera_angle} 0"/>
   </joint>
   <gazebo reference="front_camera_link">
@@ -477,5 +478,5 @@
     <parent link="rear_wagon"/>
     <child link="rear_camera_link"/>
-    <origin xyz="${rear_sensor_x} 0 ${camera_z}" rpy="0 0 3.14159"/>
+    <origin xyz="${rear_sensor_x} 0 ${camera_z}" rpy="0 ${camera_angle} ${pi}"/>
   </joint>
   <gazebo reference="rear_camera_link">

Commit message: chaged body_angle from pitch to roll

File: src/robot_description/src/urdf/Floribot.urdf.xacro (robot description, xacro)
@@ -87,6 +87,6 @@
     </inertial>
   </link>
-  <joint name="body_angle_pitch" type="revolute">
-    <axis xyz="0 1 0"/>
+  <joint name="body_angle_roll" type="revolute">
+    <axis xyz="1 0 0"/>
     <limit effort="1.0" lower="-1.57" upper="1.57" velocity="0.5"/>
     <parent link="axesFront"/>

Commit message: inserted base_footprint

File: src/robot_description/src/urdf/Floribot.urdf.xacro (robot description, xacro)
@@ -24,7 +24,13 @@
   <xacro:property name="camera_angle" value="0.6" />
   <!-- <xacro:property name="pi" value="3.141592653589793" /> Muss nicht definiert werden. -->
+  <link name="base_footprint"/>
+  <joint name="base_footprint_joint" type="fixed">
+    <parent link="base_footprint"/>
+    <child link="base_link"/>
+    <origin xyz="0 0 ${wheel_radius}" rpy="0 0 0"/>
+  </joint>
   <link name="base_link">
     <visual>
-      <origin xyz="0 0 ${wheel_radius + ghost_size}" rpy="0 0 0"/>
+      <origin xyz="0 0 ${ghost_size}" rpy="0 0 0"/>
       <geometry>
         <box size="${ghost_size} ${ghost_size} ${ghost_size}"/>

Commit message: updated urdf links

File: src/robot_description/src/urdf/Floribot.urdf.xacro (robot description, xacro)
@@ -295,5 +295,5 @@
     </plugin>
   </gazebo>
-  <link name="front_laser_link">
+  <link name="sick_front_link">
     <visual>
       <origin xyz="0 0 0" rpy="0 0 0"/>
@@ -318,12 +318,12 @@
   <joint name="front_laser_joint" type="fixed">
     <parent link="axesFront"/>
-    <child link="front_laser_link"/>
+    <child link="sick_front_link"/>
     <origin xyz="${front_sensor_x} 0 ${sensor_z}" rpy="${pi} 0 0"/>
   </joint>
-  <gazebo reference="front_laser_link">
+  <gazebo reference="sick_front_link">
     <sensor name="front_laser" type="gpu_lidar">
       <pose>0 0 0 0 0 0</pose>
       <topic>/sensors/scan_front</topic>
-      <gz_frame_id>front_laser_link</gz_frame_id>
+      <gz_frame_id>sick_front_link</gz_frame_id>
       <update_rate>10</update_rate>
       <always_on>true</always_on>
@@ -351,5 +351,5 @@
     </sensor>
   </gazebo>
-  <link name="rear_laser_link">
+  <link name="sick_rear_link">
     <visual>
       <origin xyz="0 0 0" rpy="0 0 0"/>
@@ -374,12 +374,12 @@
   <joint name="rear_laser_joint" type="fixed">
     <parent link="axesRear"/>
-    <child link="rear_laser_link"/>
+    <child link="sick_rear_link"/>
     <origin xyz="${rear_sensor_x} 0 ${sensor_z}" rpy="${pi} 0 ${pi}"/>
   </joint>
-  <gazebo reference="rear_laser_link">
+  <gazebo reference="sick_rear_link">
     <sensor name="rear_laser" type="gpu_lidar">
       <pose>0 0 0 0 0 0</pose>
       <topic>/sensors/scan_rear</topic>
-      <gz_frame_id>rear_laser_link</gz_frame_id>
+      <gz_frame_id>sick_rear_link</gz_frame_id>
       <update_rate>10</update_rate>
       <always_on>true</always_on>

Commit message: added pi

File: src/robot_description/src/urdf/Floribot.urdf.xacro (robot description, xacro)
@@ -23,5 +23,5 @@
   <xacro:property name="camera_z" value="0.263" />
   <xacro:property name="camera_angle" value="0.6" />
-  <!-- <xacro:property name="pi" value="3.141592653589793" /> Muss nicht definiert werden. -->
+  <xacro:property name="pi" value="3.141592653589793" />
   <link name="base_footprint"/>
   <joint name="base_footprint_joint" type="fixed">

Commit message: Refactor joint definitions in URDF: reorder base_footprint_joint and change body_angle_roll to fixed type

File: src/robot_description/src/urdf/Floribot.urdf.xacro (robot description, xacro)
@@ -25,4 +25,15 @@
   <xacro:property name="pi" value="3.141592653589793" />
   <link name="base_footprint"/>
+  <link name="base_link">
+    <visual>
+      <origin xyz="0 0 ${ghost_size}" rpy="0 0 0"/>
+      <geometry>
+        <box size="${ghost_size} ${ghost_size} ${ghost_size}"/>
+      </geometry>
+      <material name="base_mat">
+        <color rgba="0.0 0.8 0.8 1.0"/>
+      </material>
+    </visual>
+  </link>
   <joint name="base_footprint_joint" type="fixed">
     <parent link="base_footprint"/>
@@ -30,15 +41,4 @@
     <origin xyz="0 0 ${wheel_radius}" rpy="0 0 0"/>
   </joint>
-  <link name="base_link">
-    <visual>
-      <origin xyz="0 0 ${ghost_size}" rpy="0 0 0"/>
-      <geometry>
-        <box size="${ghost_size} ${ghost_size} ${ghost_size}"/>
-      </geometry>
-      <material name="base_mat">
-        <color rgba="0.0 0.8 0.8 1.0"/>
-      </material>
-    </visual>
-  </link>
   <link name="axesFront"/>
   <joint name="base_link_2_axesFront" type="fixed">
@@ -93,5 +93,5 @@
     </inertial>
   </link>
-  <joint name="body_angle_roll" type="revolute">
+  <joint name="body_angle_roll" type="fixed">
     <axis xyz="1 0 0"/>
     <limit effort="1.0" lower="-1.57" upper="1.57" velocity="0.5"/>

Commit message: Add IMU link and joint to URDF with offset properties

File: src/robot_description/src/urdf/Floribot.urdf.xacro (robot description, xacro)
@@ -24,4 +24,7 @@
   <xacro:property name="camera_angle" value="0.6" />
   <xacro:property name="pi" value="3.141592653589793" />
+  <xacro:property name="imu_offset_x" value="0.0" />
+  <xacro:property name="imu_offset_y" value="0.0" />
+  <xacro:property name="imu_offset_z" value="${wheel_radius + height_wagon/2}" />
   <link name="base_footprint"/>
   <link name="base_link">
@@ -394,3 +397,22 @@
     <origin xyz="${rear_sensor_x} 0 ${camera_z}" rpy="0 ${camera_angle} ${pi}"/>
   </joint>
+  <link name="imu_link">
+    <visual>
+      <geometry>
+        <box size="0.039 0.042 0.028"/>
+      </geometry>
+      <material name="imu_mat">
+        <color rgba="1.0 0.0 0.0 1.0"/>
+      </material>
+    </visual>
+    <inertial>
+      <mass value="0.01"/>
+      <inertia ixx="0.000001" ixy="0.0" ixz="0.0" iyy="0.000001" iyz="0.0" izz="0.000001"/>
+    </inertial>
+  </link>
+  <joint name="imu_joint" type="fixed">
+    <parent link="base_link"/>
+    <child link="imu_link"/>
+    <origin xyz="${imu_offset_x} ${imu_offset_y} ${imu_offset_z}" rpy="${pi} 0 ${pi}"/>
+  </joint>
 </robot>

Commit message: Rename camera and IMU links for clarity: front_camera_link to realsense_front_link, rear_camera_link to realsense_rear_link, and imu_link to xsens_mti_link

File: src/robot_description/src/urdf/Floribot.urdf.xacro (robot description, xacro)
@@ -345,5 +345,5 @@
     <origin xyz="${rear_sensor_x} 0 ${sensor_z}" rpy="${pi} 0 ${pi}"/>
   </joint>
-  <link name="front_camera_link">
+  <link name="realsense_front_link">
     <visual>
       <origin xyz="0 0 0" rpy="0 0 0"/>
@@ -368,8 +368,8 @@
   <joint name="front_camera_joint" type="fixed">
     <parent link="base_link"/>
-    <child link="front_camera_link"/>
+    <child link="realsense_front_link"/>
     <origin xyz="${front_sensor_x} 0 ${camera_z}" rpy="0 ${camera_angle} 0"/>
   </joint>
-  <link name="rear_camera_link">
+  <link name="realsense_rear_link">
     <visual>
       <origin xyz="0 0 0" rpy="0 0 0"/>
@@ -394,8 +394,8 @@
   <joint name="rear_camera_joint" type="fixed">
     <parent link="rear_wagon"/>
-    <child link="rear_camera_link"/>
+    <child link="realsense_rear_link"/>
     <origin xyz="${rear_sensor_x} 0 ${camera_z}" rpy="0 ${camera_angle} ${pi}"/>
   </joint>
-  <link name="imu_link">
+  <link name="xsens_mti_link"> <!-- Link for IMU Sensor -->
     <visual>
       <geometry>
@@ -413,5 +413,5 @@
   <joint name="imu_joint" type="fixed">
     <parent link="base_link"/>
-    <child link="imu_link"/>
+    <child link="xsens_mti_link"/>
     <origin xyz="${imu_offset_x} ${imu_offset_y} ${imu_offset_z}" rpy="${pi} 0 ${pi}"/>
   </joint>

Commit message: Fix IMU offset and joint orientation in URDF: set imu_offset_z to a fixed value and adjust rpy for imu_joint

File: src/robot_description/src/urdf/Floribot.urdf.xacro (robot description, xacro)
@@ -26,5 +26,5 @@
   <xacro:property name="imu_offset_x" value="0.0" />
   <xacro:property name="imu_offset_y" value="0.0" />
-  <xacro:property name="imu_offset_z" value="${wheel_radius + height_wagon/2}" />
+  <xacro:property name="imu_offset_z" value="0.27" />
   <link name="base_footprint"/>
   <link name="base_link">
@@ -414,5 +414,5 @@
     <parent link="base_link"/>
     <child link="xsens_mti_link"/>
-    <origin xyz="${imu_offset_x} ${imu_offset_y} ${imu_offset_z}" rpy="${pi} 0 ${pi}"/>
+    <origin xyz="${imu_offset_x} ${imu_offset_y} ${imu_offset_z}" rpy="${pi} 0 0"/>
   </joint>
 </robot>

Commit message: drehe imu in tf

File: src/robot_description/src/urdf/Floribot.urdf.xacro (robot description, xacro)
@@ -414,5 +414,5 @@
     <parent link="base_link"/>
     <child link="xsens_mti_link"/>
-    <origin xyz="${imu_offset_x} ${imu_offset_y} ${imu_offset_z}" rpy="${pi} 0 0"/>
+    <origin xyz="${imu_offset_x} ${imu_offset_y} ${imu_offset_z}" rpy="${pi} 0 ${pi}"/>
   </joint>
 </robot>

Commit message: removed rotation around z of imu_frame

File: src/robot_description/src/urdf/Floribot.urdf.xacro (robot description, xacro)
@@ -414,5 +414,5 @@
     <parent link="base_link"/>
     <child link="xsens_mti_link"/>
-    <origin xyz="${imu_offset_x} ${imu_offset_y} ${imu_offset_z}" rpy="${pi} 0 ${pi}"/>
+    <origin xyz="${imu_offset_x} ${imu_offset_y} ${imu_offset_z}" rpy="${pi} 0 0"/>
   </joint>
 </robot>

Commit message: Mehrlinienlaser als robosense_link im urdf vorbereitet

File: src/robot_description/src/urdf/Floribot.urdf.xacro (robot description, xacro)
@@ -27,4 +27,10 @@
   <xacro:property name="imu_offset_y" value="0.0" />
   <xacro:property name="imu_offset_z" value="0.27" />
+  <xacro:property name="robosense_offset_x" value="0.0" />
+  <xacro:property name="robosense_offset_y" value="0.0" />
+  <xacro:property name="robosense_offset_z" value="0.0" />
+  <xacro:property name="robosense_roll" value="0.0" />
+  <xacro:property name="robosense_pitch" value="0.0" />
+  <xacro:property name="robosense_yaw" value="0.0" />
   <link name="base_footprint"/>
   <link name="base_link">
@@ -397,4 +403,30 @@
     <origin xyz="${rear_sensor_x} 0 ${camera_z}" rpy="0 ${camera_angle} ${pi}"/>
   </joint>
+  <link name="robosense_link">
+    <visual>
+      <origin xyz="0 0 0" rpy="0 0 0"/>
+      <geometry>
+        <cylinder length="0.08" radius="0.055"/>
+      </geometry>
+      <material name="robosense_mat">
+        <color rgba="0.05 0.05 0.05 1.0"/>
+      </material>
+    </visual>
+    <collision>
+      <origin xyz="0 0 0" rpy="0 0 0"/>
+      <geometry>
+        <cylinder length="0.08" radius="0.055"/>
+      </geometry>
+    </collision>
+    <inertial>
+      <mass value="0.5"/>
+      <inertia ixx="0.0005" ixy="0.0" ixz="0.0" iyy="0.0005" iyz="0.0" izz="0.0005"/>
+    </inertial>
+  </link>
+  <joint name="robosense_joint" type="fixed">
+    <parent link="base_link"/>
+    <child link="robosense_link"/>
+    <origin xyz="${robosense_offset_x} ${robosense_offset_y} ${robosense_offset_z}" rpy="${robosense_roll} ${robosense_pitch} ${robosense_yaw}"/>
+  </joint>
   <link name="xsens_mti_link"> <!-- Link for IMU Sensor -->
     <visual>

Commit message: changed robosense link name

File: src/robot_description/src/urdf/Floribot.urdf.xacro (robot description, xacro)
@@ -403,5 +403,5 @@
     <origin xyz="${rear_sensor_x} 0 ${camera_z}" rpy="0 ${camera_angle} ${pi}"/>
   </joint>
-  <link name="robosense_link">
+  <link name="rslidar">
     <visual>
       <origin xyz="0 0 0" rpy="0 0 0"/>
@@ -426,5 +426,5 @@
   <joint name="robosense_joint" type="fixed">
     <parent link="base_link"/>
-    <child link="robosense_link"/>
+    <child link="rslidar"/>
     <origin xyz="${robosense_offset_x} ${robosense_offset_y} ${robosense_offset_z}" rpy="${robosense_roll} ${robosense_pitch} ${robosense_yaw}"/>
   </joint>

Commit message: Update Floribot.urdf.xacro edited parameters robosense

File: src/robot_description/src/urdf/Floribot.urdf.xacro (robot description, xacro)
@@ -27,9 +27,9 @@
   <xacro:property name="imu_offset_y" value="0.0" />
   <xacro:property name="imu_offset_z" value="0.27" />
-  <xacro:property name="robosense_offset_x" value="0.0" />
+  <xacro:property name="robosense_offset_x" value="0.225" />
   <xacro:property name="robosense_offset_y" value="0.0" />
-  <xacro:property name="robosense_offset_z" value="0.0" />
+  <xacro:property name="robosense_offset_z" value="0.815" />
   <xacro:property name="robosense_roll" value="0.0" />
-  <xacro:property name="robosense_pitch" value="0.0" />
+  <xacro:property name="robosense_pitch" value="20.0" />
   <xacro:property name="robosense_yaw" value="0.0" />
   <link name="base_footprint"/>

Commit message: Update Floribot.urdf.xacro

File: src/robot_description/src/urdf/Floribot.urdf.xacro (robot description, xacro)
@@ -30,6 +30,6 @@
   <xacro:property name="robosense_offset_y" value="0.0" />
   <xacro:property name="robosense_offset_z" value="0.815" />
-  <xacro:property name="robosense_roll" value="0.0" />
-  <xacro:property name="robosense_pitch" value="20.0" />
+  <xacro:property name="robosense_roll" value="180.0" />
+  <xacro:property name="robosense_pitch" value="-20.0" />
   <xacro:property name="robosense_yaw" value="0.0" />
   <link name="base_footprint"/>

Commit message: Update Floribot.urdf.xacro

File: src/robot_description/src/urdf/Floribot.urdf.xacro (robot description, xacro)
@@ -30,6 +30,6 @@
   <xacro:property name="robosense_offset_y" value="0.0" />
   <xacro:property name="robosense_offset_z" value="0.815" />
-  <xacro:property name="robosense_roll" value="180.0" />
-  <xacro:property name="robosense_pitch" value="-20.0" />
+  <xacro:property name="robosense_roll" value="1.57079632679" />
+  <xacro:property name="robosense_pitch" value="-0.3490658503989" />
   <xacro:property name="robosense_yaw" value="0.0" />
   <link name="base_footprint"/>

Commit message: Update robosense roll property to use pi variable

File: src/robot_description/src/urdf/Floribot.urdf.xacro (robot description, xacro)
@@ -30,5 +30,5 @@
   <xacro:property name="robosense_offset_y" value="0.0" />
   <xacro:property name="robosense_offset_z" value="0.815" />
-  <xacro:property name="robosense_roll" value="1.57079632679" />
+  <xacro:property name="robosense_roll" value="${pi}" />
   <xacro:property name="robosense_pitch" value="-0.3490658503989" />
   <xacro:property name="robosense_yaw" value="0.0" />

Commit message: kp was imu da macht

File: src/robot_description/src/urdf/Floribot.urdf.xacro (robot description, xacro)
@@ -446,5 +446,5 @@
     <parent link="base_link"/>
     <child link="xsens_mti_link"/>
-    <origin xyz="${imu_offset_x} ${imu_offset_y} ${imu_offset_z}" rpy="${pi} 0 0"/>
+    <origin xyz="${imu_offset_x} ${imu_offset_y} ${imu_offset_z}" rpy="$0 0 0"/>
   </joint>
 </robot>

Commit message: Floribot.urdf.xacro aktualisieren

File: src/robot_description/src/urdf/Floribot.urdf.xacro (robot description, xacro)
@@ -446,5 +446,5 @@
     <parent link="base_link"/>
     <child link="xsens_mti_link"/>
-    <origin xyz="${imu_offset_x} ${imu_offset_y} ${imu_offset_z}" rpy="$0 0 0"/>
+    <origin xyz="${imu_offset_x} ${imu_offset_y} ${imu_offset_z}" rpy="0 0 0"/>
   </joint>
 </robot>

Commit message: Update imu_joint origin to include roll and yaw angles

File: src/robot_description/src/urdf/Floribot.urdf.xacro (robot description, xacro)
@@ -446,5 +446,5 @@
     <parent link="base_link"/>
     <child link="xsens_mti_link"/>
-    <origin xyz="${imu_offset_x} ${imu_offset_y} ${imu_offset_z}" rpy="0 0 0"/>
+    <origin xyz="${imu_offset_x} ${imu_offset_y} ${imu_offset_z}" rpy="${pi} 0 ${pi}"/>
   </joint>
 </robot>

Commit message: Fix imu_joint origin to correct roll angle and update odom0_config settings

File: src/robot_description/src/urdf/Floribot.urdf.xacro (robot description, xacro)
@@ -446,5 +446,5 @@
     <parent link="base_link"/>
     <child link="xsens_mti_link"/>
-    <origin xyz="${imu_offset_x} ${imu_offset_y} ${imu_offset_z}" rpy="${pi} 0 ${pi}"/>
+    <origin xyz="${imu_offset_x} ${imu_offset_y} ${imu_offset_z}" rpy="${pi} 0 0"/>
   </joint>
 </robot>

Commit message: Update Floribot.urdf.xacro added gps link

File: src/robot_description/src/urdf/Floribot.urdf.xacro (robot description, xacro)
@@ -33,4 +33,7 @@
   <xacro:property name="robosense_pitch" value="-0.3490658503989" />
   <xacro:property name="robosense_yaw" value="0.0" />
+  <xacro:property name="gps_offset_x" value="${imu_offset_x}" />
+  <xacro:property name="gps_offset_y" value="${imu_offset_y}" />
+  <xacro:property name="gps_offset_z" value="${imu_offset_z + 0.02}" />
   <link name="base_footprint"/>
   <link name="base_link">
@@ -448,3 +451,32 @@
     <origin xyz="${imu_offset_x} ${imu_offset_y} ${imu_offset_z}" rpy="${pi} 0 0"/>
   </joint>
+  <link name="gps_link">
+    <visual>
+      <origin xyz="0 0 0" rpy="0 0 0"/>
+      <geometry>
+        <cylinder length="0.035" radius="0.045"/>
+      </geometry>
+      <material name="gps_mat">
+        <color rgba="0.0 0.2 1.0 1.0"/>
+      </material>
+    </visual>
+    <collision>
+      <origin xyz="0 0 0" rpy="0 0 0"/>
+      <geometry>
+        <cylinder length="0.035" radius="0.045"/>
+      </geometry>
+    </collision>
+    <inertial>
+      <mass value="0.05"/>
+      <inertia
+        ixx="0.00001" ixy="0.0" ixz="0.0"
+        iyy="0.00001" iyz="0.0"
+        izz="0.00001"/>
+    </inertial>
+  </link>
+  <joint name="gps_joint" type="fixed">
+    <parent link="base_link"/>
+    <child link="gps_link"/>
+    <origin xyz="${gps_offset_x} ${gps_offset_y} ${gps_offset_z}" rpy="0 0 0"/>
+  </joint>
 </robot>

Commit message: Update Floribot.urdf.xacro

File: src/robot_description/src/urdf/Floribot.urdf.xacro (robot description, xacro)
@@ -453,5 +453,5 @@
   <link name="gps_link">
     <visual>
-      <origin xyz="0 0 0" rpy="0 0 0"/>
+      <origin xyz="-0.06 0 0" rpy="0 0 0"/>
       <geometry>
         <cylinder length="0.035" radius="0.045"/>
