Commit message: added robosense_rear_link

File: src/robot_description/src/urdf/Floribot.urdf.xacro (robot description, xacro)
@@ -33,4 +33,10 @@
   <xacro:property name="robosense_pitch" value="-0.3490658503989" />
   <xacro:property name="robosense_yaw" value="0.0" />
+  <xacro:property name="robosense_offset_rear_x" value="-0.225" />
+  <xacro:property name="robosense_offset_rear_y" value="0.0" />
+  <xacro:property name="robosense_offset_rear_z" value="0.815" />
+  <xacro:property name="robosense_rear_roll" value="${pi}" />
+  <xacro:property name="robosense_rear_pitch" value="-0.3490658503989" />
+  <xacro:property name="robosense_rear_yaw" value="${pi}" />
   <xacro:property name="gps_offset_x" value="${imu_offset_x}" />
   <xacro:property name="gps_offset_y" value="${imu_offset_y}" />
@@ -406,5 +412,5 @@
     <origin xyz="${rear_sensor_x} 0 ${camera_z}" rpy="0 ${camera_angle} ${pi}"/>
   </joint>
-  <link name="rslidar">
+  <link name="robosense_front_link">
     <visual>
       <origin xyz="0 0 0" rpy="0 0 0"/>
@@ -427,8 +433,34 @@
     </inertial>
   </link>
-  <joint name="robosense_joint" type="fixed">
+  <joint name="robosense_front_joint" type="fixed">
     <parent link="base_link"/>
-    <child link="rslidar"/>
+    <child link="robosense_front_link"/>
     <origin xyz="${robosense_offset_x} ${robosense_offset_y} ${robosense_offset_z}" rpy="${robosense_roll} ${robosense_pitch} ${robosense_yaw}"/>
+  </joint>
+  <link name="robosense_rear_link">
+    <visual>
+      <origin xyz="0 0 0" rpy="0 0 0"/>
+      <geometry>
+        <cylinder length="0.08" radius="0.055"/>
+      </geometry>
+      <material name="robosense_mat">
+        <color rgba="0.05 0.05 0.05 1.0"/>
+      </material>
+    </visual>
+    <collision>
+      <origin xyz="0 0 0" rpy="0 0 0"/>
+      <geometry>
+        <cylinder length="0.08" radius="0.055"/>
+      </geometry>
+    </collision>
+    <inertial>
+      <mass value="0.5"/>
+      <inertia ixx="0.0005" ixy="0.0" ixz="0.0" iyy="0.0005" iyz="0.0" izz="0.0005"/>
+    </inertial>
+  </link>
+  <joint name="robosense_rear_joint" type="fixed">
+    <parent link="axesRear"/>
+    <child link="robosense_rear_link"/>
+    <origin xyz="${robosense_offset_rear_x} ${robosense_offset_rear_y} ${robosense_offset_rear_z}" rpy="${robosense_rear_roll} ${robosense_rear_pitch} ${robosense_rear_yaw}"/>
   </joint>
   <link name="xsens_mti_link"> <!-- Link for IMU Sensor -->

Commit message: Update robosense rear properties for improved sensor alignment

File: src/robot_description/src/urdf/Floribot.urdf.xacro (robot description, xacro)
@@ -37,6 +37,6 @@
   <xacro:property name="robosense_offset_rear_z" value="0.815" />
   <xacro:property name="robosense_rear_roll" value="${pi}" />
-  <xacro:property name="robosense_rear_pitch" value="-0.3490658503989" />
-  <xacro:property name="robosense_rear_yaw" value="${pi}" />
+  <xacro:property name="robosense_rear_pitch" value="2.79253" />
+  <xacro:property name="robosense_rear_yaw" value="0.0" />
   <xacro:property name="gps_offset_x" value="${imu_offset_x}" />
   <xacro:property name="gps_offset_y" value="${imu_offset_y}" />

Commit message: Update robosense rear properties for improved sensor calibration

File: src/robot_description/src/urdf/Floribot.urdf.xacro (robot description, xacro)
@@ -37,6 +37,6 @@
   <xacro:property name="robosense_offset_rear_z" value="0.815" />
   <xacro:property name="robosense_rear_roll" value="${pi}" />
-  <xacro:property name="robosense_rear_pitch" value="2.79253" />
-  <xacro:property name="robosense_rear_yaw" value="0.0" />
+  <xacro:property name="robosense_rear_pitch" value="-0.3490658503989" />
+  <xacro:property name="robosense_rear_yaw" value="${pi}" />
   <xacro:property name="gps_offset_x" value="${imu_offset_x}" />
   <xacro:property name="gps_offset_y" value="${imu_offset_y}" />

Commit message: Add axesRear_footprint link and joint for improved robot structure

File: src/robot_description/src/urdf/Floribot.urdf.xacro (robot description, xacro)
@@ -173,4 +173,31 @@
     <origin xyz="${-wheel_joint_2_mid_joint + vertical_length/2} 0 0"/>
   </joint>
+  <link name="axesRear_footprint">
+    <visual>
+      <origin xyz="0 0 0" rpy="0 0 0"/>
+      <geometry>
+        <box size="${ghost_size} ${ghost_size} ${ghost_size}"/>
+      </geometry>
+      <material name="axes_rear_footprint_mat">
+        <color rgba="0.8 0 0.8 1.0"/>
+      </material>
+    </visual>
+    <collision>
+      <origin xyz="0 0 0" rpy="0 0 0"/>
+      <geometry>
+        <box size="${ghost_size} ${ghost_size} ${ghost_size}"/>
+      </geometry>
+    </collision>
+    <inertial>
+      <origin xyz="0 0 0" rpy="0 0 0"/>
+      <mass value="0.001"/>
+      <inertia ixx="1.369982" ixy="0.0" ixz="0.0" iyy="0.487502" iyz="0.0" izz="1.132200"/>
+    </inertial>
+  </link>
+  <joint name="j_axesRear_2_axesRear_footprint" type="fixed">
+    <parent link="axesRear"/>
+    <child link="axesRear_footprint"/>
+    <origin xyz="0.0 0.0 -${wheel_radius}" rpy="0 0 ${pi}"/>
+  </joint>
   <joint name="j_axesRear_2_rear_wagon" type="fixed">
     <parent link="axesRear"/>

Commit message: Update rear camera properties and joint configuration for improved sensor integration

File: src/robot_description/src/urdf/Floribot.urdf.xacro (robot description, xacro)
@@ -24,4 +24,8 @@
   <xacro:property name="camera_angle" value="0.6" />
   <xacro:property name="pi" value="3.141592653589793" />
+  <xacro:property name="camera_x_rear" value="0.275" />
+  <xacro:property name="camera_y_rear" value="0.035" />
+  <xacro:property name="camera_z_rear" value="0.825" />
+  <xacro:property name="camera_angle_rear" value="0.785398" />
   <xacro:property name="imu_offset_x" value="0.0" />
   <xacro:property name="imu_offset_y" value="0.0" />
@@ -413,5 +417,5 @@
     <origin xyz="${front_sensor_x} 0 ${camera_z}" rpy="0 ${camera_angle} 0"/>
   </joint>
-  <link name="realsense_rear_link">
+  <link name="realsense_rear_link">  <!-- als REalsense oben deklariert -->
     <visual>
       <origin xyz="0 0 0" rpy="0 0 0"/>
@@ -435,7 +439,7 @@
   </link>
   <joint name="rear_camera_joint" type="fixed">
-    <parent link="rear_wagon"/>
+    <parent link="base_link"/>
     <child link="realsense_rear_link"/>
-    <origin xyz="${rear_sensor_x} 0 ${camera_z}" rpy="0 ${camera_angle} ${pi}"/>
+    <origin xyz="${camera_x_rear} ${camera_y_rear} ${camera_z_rear}" rpy="0 ${camera_angle_rear} 0"/>
   </joint>
   <link name="robosense_front_link">

Commit message: Add pan-tilt link and joint for enhanced sensor positioning

File: src/robot_description/src/urdf/Floribot.urdf.xacro (robot description, xacro)
@@ -46,4 +46,7 @@
   <xacro:property name="gps_offset_y" value="${imu_offset_y}" />
   <xacro:property name="gps_offset_z" value="${imu_offset_z + 0.02}" />
+  <xacro:property name="pan_tilt_offset_x" value="-0.23" />
+  <xacro:property name="pan_tilt_offset_y" value="-0.03" />
+  <xacro:property name="pan_tilt_offset_z" value="0.0" />
   <link name="base_footprint"/>
   <link name="base_link">
@@ -204,4 +207,31 @@
     <origin xyz="0.0 0.0 -${wheel_radius}" rpy="0 0 ${pi}"/>
   </joint>
+  <link name="pan_tilt_link_footprint">
+    <visual>
+      <origin xyz="0 0 0" rpy="0 0 0"/>
+      <geometry>
+        <box size="${ghost_size} ${ghost_size} ${ghost_size}"/>
+      </geometry>
+      <material name="pan_tilt_footprint_mat">
+        <color rgba="0.8 0.8 0 1.0"/>
+      </material>
+    </visual>
+    <collision>
+      <origin xyz="0 0 0" rpy="0 0 0"/>
+      <geometry>
+        <box size="${ghost_size} ${ghost_size} ${ghost_size}"/>
+      </geometry>
+    </collision>
+    <inertial>
+      <origin xyz="0 0 0" rpy="0 0 0"/>
+      <mass value="0.001"/>
+      <inertia ixx="0.000001" ixy="0.0" ixz="0.0" iyy="0.000001" iyz="0.0" izz="0.000001"/>
+    </inertial>
+  </link>
+  <joint name="pan_tilt_link_footprint_joint" type="fixed">
+    <parent link="axesRear_footprint"/>
+    <child link="pan_tilt_link_footprint"/>
+    <origin xyz="${pan_tilt_offset_x} ${pan_tilt_offset_y} ${pan_tilt_offset_z}" rpy="0 0 ${pi}"/>
+  </joint>
   <joint name="j_axesRear_2_rear_wagon" type="fixed">
     <parent link="axesRear"/>
